File: Departement/Elektrotekniska/circuit/bryggan_motherboard/bryggan_motherboard.kicad_pcb (KiCad board)
At the start: 2 copper layers, 65 x 56.5 mm, 14 parts, among them J1 RJ12, J2 Screw_Terminal_01x07, J3 Barrel_Jack, P3 Raspberry_Pi_+_Conn, Q1 BSS138, U1 ULN2003A, U5 DMMT5401

Commit message: fine lire
Routing:
- removed copper zone on B.Cu, net GND
Changed lines of the file:
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@@
   )
   (setup
-    (last_trace_width 0.6)
+    (last_trace_width 1)
     (user_trace_width 0.1)
     (user_trace_width 0.2)
@@
   (gr_arc (start 166.92 74.07) (end 166.92 71.07) (angle 90) (layer Edge.Cuts) (width 0.1))
   (gr_arc (start 107.92 124.57) (end 107.92 127.57) (angle 90) (layer Edge.Cuts) (width 0.1))
-  (segment (start 113.31 73.76) (end 112.04 73.76) (width 0.6) (layer F.Cu) (net 2))
-  (segment (start 121.14336 80.32336) (end 121.14336 86.46) (width 0.6) (layer F.Cu) (net 2))
-  (segment (start 119.66 78.84) (end 121.14336 80.32336) (width 0.6) (layer F.Cu) (net 2))
-  (segment (start 110.77 78.84) (end 119.66 78.84) (width 0.6) (layer F.Cu) (net 2))
-  (segment (start 110.77 75.03) (end 110.77 78.84) (width 0.6) (layer F.Cu) (net 2))
-  (segment (start 112.04 73.76) (end 110.77 75.03) (width 0.6) (layer F.Cu) (net 2))
-  (segment (start 115.85 73.76) (end 113.31 73.76) (width 0.6) (layer F.Cu) (net 2))
+  (segment (start 113.31 73.76) (end 112.04 73.76) (width 1) (layer F.Cu) (net 2))
+  (segment (start 112.04 73.76) (end 110.77 75.03) (width 1) (layer F.Cu) (net 2))
+  (segment (start 110.77 75.03) (end 110.77 78.84) (width 1) (layer F.Cu) (net 2))
+  (segment (start 110.77 78.84) (end 119.66 78.84) (width 1) (layer F.Cu) (net 2))
+  (segment (start 119.66 78.84) (end 121.14336 80.32336) (width 1) (layer F.Cu) (net 2))
+  (segment (start 121.14336 80.32336) (end 121.14336 86.46) (width 1) (layer F.Cu) (net 2))
+  (segment (start 115.85 73.76) (end 113.31 73.76) (width 1) (layer F.Cu) (net 2))
   (segment (start 122.2 89.21336) (end 122.2 87.73) (width 0.6) (layer F.Cu) (net 2))
   (segment (start 122.2 87.73) (end 120.93 86.46) (width 0.6) (layer F.Cu) (net 2))
   (segment (start 120.93 86.46) (end 121.14336 86.46) (width 0.6) (layer F.Cu) (net 2))
-  (segment (start 143.79 100.43) (end 143.79 90.27) (width 0.6) (layer F.Cu) (net 3))
-  (segment (start 150.14 122.02) (end 150.14 106.78) (width 0.6) (layer F.Cu) (net 3))
-  (segment (start 150.14 106.78) (end 143.79 100.43) (width 0.6) (layer F.Cu) (net 3))
-  (segment (start 148.87 123.29) (end 150.14 122.02) (width 0.6) (layer F.Cu) (net 3))
-  (segment (start 132.36 123.29) (end 148.87 123.29) (width 0.6) (layer F.Cu) (net 3))
-  (segment (start 124.74 115.67) (end 132.36 123.29) (width 0.6) (layer F.Cu) (net 3))
-  (segment (start 124.74 97.89) (end 124.74 115.67) (width 0.6) (layer F.Cu) (net 3))
-  (segment (start 128.8675 85.5075) (end 123.25664 85.5075) (width 0.6) (layer F.Cu) (net 3))
-  (segment (start 129.82 86.46) (end 128.8675 85.5075) (width 0.6) (layer F.Cu) (net 3))
-  (segment (start 129.82 92.81) (end 129.82 86.46) (width 0.6) (layer F.Cu) (net 3))
-  (segment (start 124.74 97.89) (end 129.82 92.81) (width 0.6) (layer F.Cu) (net 3))
+  (segment (start 143.79 100.43) (end 143.79 90.27) (width 1) (layer F.Cu) (net 3))
+  (segment (start 124.74 97.89) (end 124.74 115.67) (width 1) (layer F.Cu) (net 3))
+  (segment (start 124.74 115.67) (end 132.36 123.29) (width 1) (layer F.Cu) (net 3))
+  (segment (start 132.36 123.29) (end 148.87 123.29) (width 1) (layer F.Cu) (net 3))
+  (segment (start 148.87 123.29) (end 150.14 122.02) (width 1) (layer F.Cu) (net 3))
+  (segment (start 150.14 106.78) (end 143.79 100.43) (width 1) (layer F.Cu) (net 3))
+  (segment (start 150.14 122.02) (end 150.14 106.78) (width 1) (layer F.Cu) (net 3))
+  (segment (start 128.8675 85.5075) (end 123.25664 85.5075) (width 1) (layer F.Cu) (net 3))
+  (segment (start 124.74 97.89) (end 129.82 92.81) (width 1) (layer F.Cu) (net 3))
+  (segment (start 129.82 92.81) (end 129.82 86.46) (width 1) (layer F.Cu) (net 3))
+  (segment (start 129.82 86.46) (end 128.8675 85.5075) (width 1) (layer F.Cu) (net 3))
   (segment (start 124.74 97.89) (end 124.74 96.62) (width 0.6) (layer F.Cu) (net 3))
-  (segment (start 124.74 96.62) (end 119.66 91.54) (width 0.6) (layer F.Cu) (net 3))
-  (segment (start 119.66 90.80086) (end 121.2475 89.21336) (width 0.6) (layer F.Cu) (net 3))
-  (segment (start 119.66 91.54) (end 119.66 90.80086) (width 0.6) (layer F.Cu) (net 3))
+  (segment (start 124.74 96.62) (end 119.66 91.54) (width 1) (layer F.Cu) (net 3))
+  (segment (start 119.66 91.54) (end 119.66 90.80086) (width 1) (layer F.Cu) (net 3))
+  (segment (start 119.66 90.80086) (end 121.2475 89.21336) (width 1) (layer F.Cu) (net 3))
   (segment (start 126.3275 87.4125) (end 126.645 87.095) (width 0.6) (layer F.Cu) (net 6))
   (segment (start 123.25664 87.4125) (end 126.3275 87.4125) (width 0.6) (layer F.Cu) (net 6))
@@
   (segment (start 126.22 73.55) (end 127.28 74.61) (width 0.3) (layer F.Cu) (net 36) (status 10))
   (segment (start 146.33 80.11) (end 146.33 82.65) (width 0.3) (layer F.Cu) (net 36))
-  (segment (start 148.87 90.27) (end 148.87 96.62) (width 0.6) (layer F.Cu) (net 37))
-  (segment (start 148.87 96.62) (end 164.11 111.86) (width 0.6) (layer F.Cu) (net 37))
+  (segment (start 148.87 90.27) (end 148.87 96.62) (width 1) (layer F.Cu) (net 37))
+  (segment (start 148.87 96.62) (end 164.11 111.86) (width 1) (layer F.Cu) (net 37))
   (segment (start 164.11 111.86) (end 164.11 112.17) (width 0.5) (layer F.Cu) (net 37))
-  (segment (start 146.33 90.27) (end 146.33 97.89) (width 0.6) (layer F.Cu) (net 38))
-  (segment (start 146.33 97.89) (end 164.11 115.67) (width 0.6) (layer F.Cu) (net 38))
-  (segment (start 151.41 90.27) (end 151.41 95.97) (width 0.6) (layer F.Cu) (net 39))
-  (segment (start 151.41 95.97) (end 164.11 108.67) (width 0.6) (layer F.Cu) (net 39))
-  (segment (start 153.95 90.27) (end 153.95 95.01) (width 0.6) (layer F.Cu) (net 40))
-  (segment (start 153.95 95.01) (end 164.11 105.17) (width 0.6) (layer F.Cu) (net 40))
-  (segment (start 156.49 90.27) (end 156.49 94.05) (width 0.6) (layer F.Cu) (net 41))
-  (segment (start 156.49 94.05) (end 164.11 101.67) (width 0.6) (layer F.Cu) (net 41))
-  (segment (start 159.03 90.27) (end 159.03 93.09) (width 0.6) (layer F.Cu) (net 42))
-  (segment (start 159.03 93.09) (end 164.11 98.17) (width 0.6) (layer F.Cu) (net 42))
-  (segment (start 161.57 90.27) (end 161.57 92.13) (width 0.6) (layer F.Cu) (net 43))
-  (segment (start 161.57 92.13) (end 164.11 94.67) (width 0.6) (layer F.Cu) (net 43))
+  (segment (start 146.33 90.27) (end 146.33 97.89) (width 1) (layer F.Cu) (net 38))
+  (segment (start 146.33 97.89) (end 164.11 115.67) (width 1) (layer F.Cu) (net 38))
+  (segment (start 151.41 90.27) (end 151.41 95.97) (width 1) (layer F.Cu) (net 39))
+  (segment (start 151.41 95.97) (end 164.11 108.67) (width 1) (layer F.Cu) (net 39))
+  (segment (start 153.95 90.27) (end 153.95 95.01) (width 1) (layer F.Cu) (net 40))
+  (segment (start 153.95 95.01) (end 164.11 105.17) (width 1) (layer F.Cu) (net 40))
+  (segment (start 156.49 90.27) (end 156.49 94.05) (width 1) (layer F.Cu) (net 41))
+  (segment (start 156.49 94.05) (end 164.11 101.67) (width 1) (layer F.Cu) (net 41))
+  (segment (start 159.03 90.27) (end 159.03 93.09) (width 1) (layer F.Cu) (net 42))
+  (segment (start 159.03 93.09) (end 164.11 98.17) (width 1) (layer F.Cu) (net 42))
+  (segment (start 161.57 90.27) (end 161.57 92.13) (width 1) (layer F.Cu) (net 43))
+  (segment (start 161.57 92.13) (end 164.11 94.67) (width 1) (layer F.Cu) (net 43))
   (segment (start 128.55 73.76) (end 129.82 75.03) (width 0.5) (layer F.Cu) (net 46))
   (segment (start 129.82 75.03) (end 129.82 77.57) (width 0.5) (layer F.Cu) (net 46))
   (zone (net 1) (net_name GND) (layer F.Cu) (hatch edge 0.508)
-    (connect_pads yes (clearance 0.25))
-    (min_thickness 0.05)
-    (fill yes (arc_segments 16) (thermal_gap 0.508) (thermal_bridge_width 0.508) (smoothing fillet) (radius 1))
-    (polygon
-      (pts
-        (xy 89.66 134.09) (xy 82.66 134.09) (xy 82.66 141.09) (xy 32.16 141.09) (xy 32.16 134.09)
-        (xy 25.66 134.09) (xy 25.66 122.59) (xy 30.66 122.59) (xy 30.66 104.59) (xy 25.66 104.59)
-        (xy 25.66 92.59) (xy 32.16 92.59) (xy 32.16 85.59) (xy 83.16 85.59) (xy 83.16 92.59)
-        (xy 89.66 92.59)
-      )
-    )
-  )
-  (zone (net 1) (net_name GND) (layer B.Cu) (hatch edge 0.508)
-    (connect_pads yes (clearance 0.25))
-    (min_thickness 0.05)
-    (fill yes (arc_segments 16) (thermal_gap 0.508) (thermal_bridge_width 0.508) (smoothing fillet) (radius 1))
-    (polygon
-      (pts
-        (xy 89.66 134.09) (xy 82.66 134.09) (xy 82.66 141.09) (xy 32.16 141.09) (xy 32.16 134.09)
-        (xy 25.66 134.09) (xy 25.66 122.59) (xy 30.66 122.59) (xy 30.66 104.59) (xy 25.66 104.59)
-        (xy 25.66 92.59) (xy 32.16 92.59) (xy 32.16 85.59) (xy 83.16 85.59) (xy 83.16 92.59)
-        (xy 89.66 92.59)
-      )
-    )
-  )
-  (zone (net 1) (net_name GND) (layer F.Cu) (hatch edge 0.508)
     (connect_pads (clearance 0.508))
